File: hw/pcb/microphone/microphone.sch (EAGLE design)
At the start: 0 parts

Commit message: Add microphone board
Completed schematic and layout of microphone board. Is a similar
design to the one from TI's tidu765 app-note. Has provisions for a
more basic non-inverting amplifier design as well. Currently uses a
transimpedence amplifier.
Parts:
- added C1, C2: (no value), wedfestdress:CAP_CGB3B1X5R1A475M055AC
- added C3: (no value), wedfestdress:CAP_C1608X7R1H104K080AA
- added C4: (no value), wedfestdress:CAP_CL10A225KP8NNNC
- added C5: (no value), wedfestdress:CAP_CL10C150JB8NNNC
- added MIC1: (no value), wedfestdress:POM-5238P-R
- added R1: (no value), wedfestdress:RES_2K2_ERJ-3EKF2201V
- added R2, R3: (no value), wedfestdress:RES_10K_RC0603FR-0710KL
- added R4: (no value), wedfestdress:RES_0R_RC0603JR-070RL
- added R5: (no value), wedfestdress:RES_75K_RC0603FR-0775KL
- added R6: (no value), wedfestdress:RES_49R9_RC0603FR-0749R9L
- added R7: (no value), wedfestdress:RES_100K_RC0603FR-07100KL
- added TP1, TP2, TP3: (no value), wedfestdress:TP_1P6_MM_ROUND
- added U1: (no value), wedfestdress:MCP6241UT-E/LT
Connections:
- new net 3V3: C3.P$1, R1.P$2, R2.P$2, TP1.P1, U1.V+
- new net AMP_NEG: C5.P$1, R4.P$2, R5.P$1, U1.IN-
- new net AMP_OUT: C5.P$2, R5.P$2, R6.P$1, U1.OUT
- new net AMP_OUT_R: C4.P$1, R6.P$2
- new net GND: C2.P$1, C3.P$2, MIC1.NEG, R3.P$1, R7.P$1, TP3.P1, U1.V-
- new net MIC_OUT: C1.P$1, MIC1.POS, R1.P$1
- new net MIC_OUT_C: C1.P$2, R4.P$1
- new net REF: C2.P$2, R2.P$1, R3.P$2, U1.IN+
- new net SIGNAL_OUT: C4.P$2, R7.P$2, TP2.P1
Other:
- note added: "From TI's app-note TIDU765 http://www.ti.com/lit/ug/tidu765/tidu765.pdf"
