File: hw/pcb/pixel/pixel.sch (EAGLE design)
At the start: 0 parts

Commit message: First pass at pixel PCB
- Add some library footprints.
- First pass on schematic and layout of pixel PCB.
Parts:
- added TP1, TP2, TP3, TP4, TP5, TP6, TP7, TP8: (no value), wedfestdress:TP_1P6_MM_ROUND
- added U1: (no value), wedfestdress:APA102C
Connections:
- new net CI: TP3.P1, U1.CI
- new net CO: TP5.P1, U1.CO
- new net DI: TP2.P1, U1.DI
- new net DO: TP6.P1, U1.DO
- new net GND: TP4.P1, TP8.P1, U1.GND
- new net V+: TP1.P1, TP7.P1, U1.VCC

Commit message: Final tweaks and CAM output for all three boards
Parts:
- added TVS1, TVS2, TVS3, TVS4: (no value), wedfestdress:PESD5V0X1UB,135
Connections:
- net CI: now also TVS1.K
- net CO: now also TVS3.K
- net DI: now also TVS2.K
- net DO: now also TVS4.K
- net GND: now also TVS1.A, TVS2.A, TVS3.A, TVS4.A
Other:
- moved on the sheet: TP1, TP2, TP3, TP4, TP5, TP6, TP7, TP8
